File: hardware/pv_panel/pv_panel.kicad_sch (KiCad schematic)
At the start: 15 parts, among them J1 Conn_01x04_Pin

Commit message: first vrack at EPS
Parts:
- removed CR5, CR6: STPS1L30MF, STPS1L40MF:STMITEFLAT_STM, symbol STPS1L40MF:STPS1L30MF
- removed J1: Conn_01x04_Pin, Connector_Molex:Molex_PicoBlade_53261-0471_1x04-1MP_P1.25mm_Horizontal, symbol Connector:Conn_01x04_Pin
- added CR1: STPS1L30MF, STPS1L40MF:STMITEFLAT_STM, symbol STPS1L40MF:STPS1L30MF
- added J1: Conn_01x02_Socket, Connector_Molex:Molex_PicoBlade_53261-0271_1x02-1MP_P1.25mm_Horizontal, symbol Connector:Conn_01x02_Socket
- PV1: renamed from PV1_PLUS1; footprint SM141K10TF:Untitled -> AnySolar:Anysolar-SM141K10TF
- PV3: renamed from PV1_MINUS1; footprint SM141K10TF:Untitled -> AnySolar:Anysolar-SM141K10TF
- PV4: renamed from PV2_MINUS1; footprint SM141K10TF:Untitled -> AnySolar:Anysolar-SM141K10TF
- VP2: renamed from VP2_PLUS1; footprint SM141K10TF:Untitled -> AnySolar:Anysolar-SM141K10TF
- renumbered CR1 to CR0
Connections:
- net VPV_MINUS is gone; now on an unnamed net: CR2.2
- net GND: now also J1.1 (Pin_1); no longer VP2.2 (-)
- net at CR0.1, PV1.1 (+): now also CR1.2
- net at PV1.2 (-), VP2.1 (+): now also CR1.1
- net at CR2.1, CR3.2, PV3.1 (+): now also VP2.2 (-)
- net VPV_PLUS renamed VPV
- net VPV: now also J1.2 (Pin_2)
Other:
- moved on the sheet: CR0
